File: PCB/Kicad/Melty.kicad_pcb (KiCad board)
At the start: 2 copper layers, 64 parts, among them J1 SWD, Q1 G35N02K, Q10 G35N02K, Q11 G35N02K, Q12 G35N02K, Q13 G35N02K, Q14 G35N02K, Q2 G35N02K, Q5 G35N02K, Q6 G35N02K, Q7 G35N02K, Q8 G35N02K, Q9 G35N02K, U1 AP7375-33SA-7, U2 PJ73AL50SQ, U3 STM32F303RBTx, U4 DRV8300DRGER, U5 TSOP348xx, U6 TSOP348xx, U7 DRV8300DRGER

Commit message: Updated PCB files
updated PCB files with a semi final version of the schematic and PCB design for Oreo
Parts:
- removed U5, U6: TSOP348xx, OptoDevice:Vishay_MOLD-3Pin
- added C16: 1u, Capacitor_SMD:C_0805_2012Metric, F.Cu at (115.2, 52.8)
- added C17: 10uF, Capacitor_SMD:C_1206_3216Metric, F.Cu at (80.9, 51.0)
- added C18: 10uF, Capacitor_SMD:C_1206_3216Metric, F.Cu at (80.7, 66.5)
- added C19: 1u, Capacitor_SMD:C_0805_2012Metric, F.Cu at (122.3, 50.6)
- added C20: 1u, Capacitor_SMD:C_0805_2012Metric, F.Cu at (96.2, 81.8)
- added C21: 1u, Capacitor_SMD:C_0805_2012Metric, F.Cu at (91.6, 87.1)
- added C22: 1u, Capacitor_SMD:C_0805_2012Metric, F.Cu at (118.4, 50.6)
- added C23: 1u, Capacitor_SMD:C_0805_2012Metric, F.Cu at (94.7, 84.9)
- added C24: 10uF, Capacitor_SMD:C_1206_3216Metric, F.Cu at (80.7, 82.0)
- added C25: 10uF, Capacitor_SMD:C_1206_3216Metric, F.Cu at (131.4, 59.3)
- added C26: 10uF, Capacitor_SMD:C_1206_3216Metric, F.Cu at (131.7, 74.7)
- added C27: 10uF, Capacitor_SMD:C_1206_3216Metric, F.Cu at (131.3, 94.0)
- added C6: 10uF, Capacitor_SMD:C_1206_3216Metric, F.Cu at (122.2, 87.9)
- added C7: 10uF, Capacitor_SMD:C_0402_1005Metric, F.Cu at (118.9, 84.4)
- added J10: Conn_01x01_Female, Connector_Wire:SolderWirePad_1x01_SMD_1x2mm, B.Cu at (108.5, 60.3)
- added J11: Conn_01x02_Female, Connector_PinSocket_2.54mm:PinSocket_1x02_P2.54mm_Vertical, F.Cu at (80.8, 48.0)
- added J12: Conn_01x07_Female, Connector_PinSocket_2.00mm:PinSocket_1x07_P2.00mm_Vertical, F.Cu at (117.2, 88.5)
- added J13: Conn_01x07_Female, Connector_PinSocket_2.00mm:PinSocket_1x07_P2.00mm_Vertical, F.Cu at (115.1, 85.5)
- added J14: Conn_01x01_Female, Connector_Wire:SolderWirePad_1x01_SMD_1x2mm, F.Cu at (107.7, 77.5)
- added J15: Conn_01x01_Female, Connector_Wire:SolderWirePad_1x01_SMD_1x2mm, F.Cu at (109.9, 78.1)
- added J2: Conn_01x01_Female, Connector_Wire:SolderWirePad_1x01_SMD_1x2mm, B.Cu at (115.9, 60.3)
- added J3: Conn_01x01_Female, Connector_Wire:SolderWirePad_1x01_SMD_1x2mm, B.Cu at (109.9, 72.9)
- added J4: Conn_01x01_Female, Connector_Wire:SolderWirePad_1x01_SMD_1x2mm, B.Cu at (105.4, 71.3)
- added J5: Conn_01x01_Female, Connector_Wire:SolderWirePad_1x01_SMD_1x2mm, B.Cu at (111.3, 60.3)
- added J6: Conn_01x01_Female, Connector_Wire:SolderWirePad_1x01_SMD_1x2mm, B.Cu at (107.9, 74.9)
- added J7: Conn_01x01_Female, Connector_Wire:SolderWirePad_1x01_SMD_1x2mm, B.Cu at (103.4, 73.4)
- added J8: Conn_01x01_Female, Connector_Wire:SolderWirePad_1x01_SMD_1x2mm, B.Cu at (105.9, 76.9)
- added J9: Conn_01x01_Female, Connector_Wire:SolderWirePad_1x01_SMD_1x2mm, B.Cu at (101.4, 75.4)
- added REF**: MountingHole_3.2mm_M3, MountingHole:MountingHole_3.2mm_M3, F.Cu at (114.2, 69.6)
- added REF**: MountingHole_3.2mm_M3, MountingHole:MountingHole_3.2mm_M3, F.Cu at (95.5, 49.9)
- added REF**: OSHW-Logo2_7.3x6mm_SilkScreen, Symbol:OSHW-Logo2_7.3x6mm_SilkScreen, B.Cu at (83.7, 85.2)
- added U10: PJ73AL50SQ, Package_TO_SOT_SMD:SOT-89-3, F.Cu at (122.2, 83.9)
- added U8: NCR421UX, Package_SO:TSOP-6_1.65x3.05mm_P0.95mm, F.Cu at (103.4, 81.9)
- added Y1: Crystal, Crystal:Crystal_SMD_3225-4Pin_3.2x2.5mm, F.Cu at (92.6, 73.9)
- C2: value 10uF -> 20pF; footprint Capacitor_SMD:C_1206_3216Metric -> Capacitor_SMD:C_0402_1005Metric
- C4: value 10uF -> 20pF
- U2: value PJ73AL50SQ -> NCR421UX; footprint Package_TO_SOT_SMD:SOT-89-3 -> Package_SO:TSOP-6_1.65x3.05mm_P0.95mm
- U4, U7: footprint Package_DFN_QFN:VQFN-24-1EP_4x4mm_P0.5mm_EP2.45x2.45mm_ThermalVias -> Package_DFN_QFN:VQFN-24-1EP_4x4mm_P0.5mm_EP2.45x2.45mm
- moved R1 143.3 mm to (92.8, 62.3), turned to 135 degrees
- moved R5 134.1 mm to (113.8, 76.8), turned to -90 degrees
- moved R4 130.7 mm to (115.4, 76.8), turned to 90 degrees
- moved C1 130.4 mm to (116.4, 82.8), turned to 0 degrees
- moved L1 127.1 mm to (112.6, 80.4), turned to -90 degrees
- moved U1 126.9 mm to (116.4, 79.9), turned to 180 degrees
- moved C5 126.3 mm to (112.8, 83.3), turned to 0 degrees
- moved C3 124.8 mm to (118.9, 81.8), turned to -90 degrees
- moved R3 117.1 mm to (108.1, 71.8), turned to 45 degrees
- moved D2 117.1 mm to (109.5, 73.1), turned to 45 degrees
- moved C4 111.6 mm to (94.7, 75.9), turned to 45 degrees
- moved C2 105.9 mm to (90.6, 71.9), turned to 45 degrees
- moved U2 99.5 mm to (107.3, 81.9), turned to 90 degrees
- moved R24 35.6 mm to (122.7, 48.8), turned to 180 degrees
- moved R23 33.9 mm to (118.1, 48.8), turned to 180 degrees
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Connections:
- C2 pad 1: +BATT -> /OSC_in
- C4 pad 1: +5V -> /OSC_out
- U2 pad 1: GND -> Heading_Red
- U2 pad 2: +5V -> Red_LED_anode
- U2 pad 3: +BATT -> Red_LED_anode
- U3 pad 16: unconnected-(U3-Pad16) -> IR_top
- U3 pad 18: unconnected-(U3-Pad18) -> IR_bottom
- U3 pad 23: unconnected-(U3-Pad23) -> Heading_Green
- U3 pad 24: unconnected-(U3-Pad24) -> Heading_Red
- U3 pad 25: unconnected-(U3-Pad25) -> Heading_Blue
- U3 pad 28: unconnected-(U3-Pad28) -> VDC_sense
- U3 pad 30: C1_Vsense -> B1_Vsense
- U3 pad 34: B1_Vsense -> A1_Vsense
- U3 pad 35: A1_Vsense -> C1_Vsense
- U3 pad 38: B1_INL -> C1_INL
- U3 pad 39: B1_INH -> C1_INH
- U3 pad 41: unconnected-(U3-Pad41) -> PPM
- U3 pad 42: C1_INL -> B1_INL
- U3 pad 43: C1_INH -> B1_INH
- U3 pad 44: unconnected-(U3-Pad44) -> PWM2
- U3 pad 45: unconnected-(U3-Pad45) -> PWM3
- U3 pad 5: Net-(C6-Pad2) -> /OSC_in
- U3 pad 6: Net-(C7-Pad2) -> /OSC_out
Routing:
- net +3V3: track 21.3 -> 120.6 mm, vias 0 -> 6
- net GND: track 21.3 -> 111.5 mm, vias 1 -> 73
- net C1: track 0.00 -> 47.3 mm, vias 0 -> 2
- net +5V: track 0.00 -> 47.3 mm, vias 0 -> 1
- net B2: track 0.00 -> 41.2 mm, vias 0 -> 2
- net A2: track 0.00 -> 38.4 mm, vias 0 -> 2
- net M1_COM: track 0.00 -> 37.7 mm, vias 0 -> 2
- net B1_Vsense: track 0.00 -> 35.0 mm, vias 0 -> 2
- net B1: track 0.00 -> 32.8 mm, vias 0 -> 2
- net A1_INL: track 0.00 -> 31.9 mm, vias 0 -> 2
- net A1_INH: track 0.00 -> 31.7 mm
- net C1_Vsense: track 0.00 -> 31.1 mm, vias 0 -> 2
- net /GHB1: track 0.00 -> 27.3 mm, vias 0 -> 2
- net /GHC1: track 0.00 -> 27.1 mm, vias 0 -> 2
- net C2: track 0.00 -> 26.4 mm, vias 0 -> 3
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- added copper zone on F.Cu, net A1
- added copper zone on F.Cu, net A2
- added copper zone on F.Cu, net B2
- added copper zone on F.Cu, net C1
- added copper zone on F.Cu, net C2
Other:
- board outline added: 80 x 50 mm
- board text added: "+"
- board text added: "-"
- board text added: "OREO V1"
- board text added: "PPM"
- board text added: "PWM2"
- board text added: "PWM3"
- board text added: "SWD"
- board text added: "github.com/BTSC10/Oreo"
