File: PCB/Kicad/Melty.kicad_sch (KiCad schematic)
At the start: 85 parts, among them J1 SWD, Q1 G35N02K, Q10 G35N02K, Q11 G35N02K, Q12 G35N02K, Q13 G35N02K, Q14 G35N02K, Q15 Q_NMOS_DSG, Q2 G35N02K, Q3 OP505, Q4 OP505, Q5 G35N02K, Q6 G35N02K, Q7 G35N02K, Q8 G35N02K, Q9 G35N02K, U1 AP7375-33SA-7, U3 STM32F303RBTx, U4 DRV8300DRGER, U5 TSOP348xx, U6 TSOP348xx, U7 DRV8300DRGER, Y1 Crystal

Commit message: Updated PCB files
updated PCB files with a semi final version of the schematic and PCB design for Oreo
Parts:
- removed D1, D3, D4: Red LED, LED_SMD:LED_0603_1608Metric, symbol Device:LED_Small
- removed Q15: Q_NMOS_DSG, symbol Device:Q_NMOS_DSG
- removed Q3, Q4: OP505, symbol Device:Q_Photo_NPN
- removed R2, R20, R21: 500R, Resistor_SMD:R_0805_2012Metric, symbol Device:R_Small
- removed R8, R9: 500R, symbol Device:R_Small
- removed RV1, RV2: 1K, symbol Device:R_Potentiometer
- removed U5, U6: TSOP348xx, OptoDevice:Vishay_MOLD-3Pin, symbol Interface_Optical:TSOP348xx
- added C2, C4: 20pF, Capacitor_SMD:C_0402_1005Metric, symbol Device:C_Small
- added C24, C25, C26, C27: 10uF, Capacitor_SMD:C_1206_3216Metric, symbol Device:C_Small
- added J10, J2, J3, J4, J5, J6, J7, J8, J9: Conn_01x01_Female, Connector_Wire:SolderWirePad_1x01_SMD_1x2mm, symbol Connector:Conn_01x01_Female
- added J11: Conn_01x02_Female, Connector_PinSocket_2.54mm:PinSocket_1x02_P2.54mm_Vertical, symbol Connector:Conn_01x02_Female
- added J12, J13: Conn_01x07_Female, Connector_PinSocket_2.00mm:PinSocket_1x07_P2.00mm_Vertical, symbol Connector:Conn_01x07_Female
- added R34, R35: 50R, symbol Device:R_Small
- added U10: PJ73AL50SQ, Package_TO_SOT_SMD:SOT-89-3, symbol Regulator_Linear:LM1117-3.3
- added U2, U8: NCR421UX, Package_SO:TSOP-6_1.65x3.05mm_P0.95mm, symbol New_Library:NCR421UX
- C14: value 100uF -> 10uF
- C16, C19, C20, C21, C22, C23: footprint (none) -> Capacitor_SMD:C_0805_2012Metric
- C17, C18: value 100n -> 10uF; footprint (none) -> Capacitor_SMD:C_1206_3216Metric
- C6: value C_Small -> 10uF; footprint (none) -> Capacitor_SMD:C_1206_3216Metric
- C7: value C_Small -> 10uF; footprint (none) -> Capacitor_SMD:C_0402_1005Metric
- U4, U7: footprint Package_DFN_QFN:VQFN-24-1EP_4x4mm_P0.5mm_EP2.45x2.45mm_ThermalVias -> Package_DFN_QFN:VQFN-24-1EP_4x4mm_P0.5mm_EP2.45x2.45mm
- Y1: footprint (none) -> Crystal:Crystal_SMD_3225-4Pin_3.2x2.5mm
Connections:
- net +3V3: now also J12.5 (Pin_5), J13.5 (Pin_5)
- net +BATT: now also C17.1, C18.1, C6.1, C24.1, C25.1, C26.1, C27.1, J11.2 (Pin_2), J12.1 (Pin_1), J12.2 (Pin_2), U10.3 (VI)
- net A1_Vsense: now also U3.34 (PB13); no longer U3.35 (PB14)
- net B1_INH: now also U3.43 (PA10); no longer U3.39 (PC8)
- net B1_INL: now also U3.42 (PA9); no longer U3.38 (PC7)
- net B1_Vsense: now also U3.30 (PB11); no longer U3.34 (PB13)
- net C1_INH: now also U3.39 (PC8); no longer U3.43 (PA10)
- net C1_INL: now also U3.38 (PC7); no longer U3.42 (PA9)
- net C1_Vsense: now also U3.35 (PB14); no longer U3.30 (PB11)
- net GND: now also C6.2, C7.2, C2.2, C24.2, C25.2, C26.2, C27.2, C4.2, J10.1 (Pin_1), J11.1 (Pin_1), J12.7 (Pin_7), J13.7 (Pin_7), J8.1 (Pin_1), J9.1 (Pin_1), R34.2, R35.2, U10.1 (GND), U2.4 (GND), U8.4 (GND); no longer C6.1, C7.1
- net IR_bottom: now also U3.18 (PF4), J13.6 (Pin_6)
- net IR_top: now also U3.16 (PA2), J12.6 (Pin_6)
- net VDC_sense: now also U3.28 (PB2)
- net OSC_in: now reaches U3.5 (PF0), Y1.1
- net OSC_in: now also C2.1; no longer C6.2
- net Heading_Green: now reaches U3.23 (PA7)
- net Heading_Green: now also U8.1 (VEN)
- net Heading_Red: now reaches U3.24 (PC4)
- net Heading_Red: now also U2.1 (VEN)
- net Heading_Blue: now reaches U3.25 (PC5)
- net PPM: now reaches U3.41 (PA8)
- net PPM: now also J5.1 (Pin_1)
- net PWM2: now reaches U3.44 (PA11)
- net PWM2: now also J6.1 (Pin_1)
- net PWM3: now reaches U3.45 (PA12)
- net PWM3: now also J7.1 (Pin_1)
- new net: J12.3 (Pin_3), J13.1 (Pin_1)
- new net: J12.4 (Pin_4), J13.2 (Pin_2)
- new net +5V: C7.1, J2.1 (Pin_1), J3.1 (Pin_1), J4.1 (Pin_1), U10.2 (VO)
- new net G_REXT: R35.1, U8.6 (REXT)
- new net Green_LED_anode: J13.4 (Pin_4), U8.2 (IOUT), U8.3 (IOUT), U8.5 (IOUT)
- new net OSC_out: C4.1, U3.6 (PF1), Y1.3
- new net R_REXT: R34.1, U2.6 (REXT)
- new net Red_LED_anode: J13.3 (Pin_3), U2.2 (IOUT), U2.3 (IOUT), U2.5 (IOUT)
- no-connect marks 11 -> 9
Other:
- note added: "300mA"
- note added: "To Daughter Boards"
- note added: "approx 20mA open = 12mA, 30R = 40mA"
- note added: "~10pF pin & board capacitance 20pF load capacitance"
- note removed: "10 mA @ 10 mW/cm2 so 330 ohms"
- moved on the sheet: AC1, C14, C15, D2, J1, R3, R4, R5
